Commit message: ran onshape

File: cybertruck_description/cybertruck/robot.urdf (robot description, URDF)
Before this commit: robot cybertruck_robot, 1 links, 0 joints
Links:
- added link part_2, mass 0.018932239501192930919; collision mesh filename=package://cybertruck_description/cybertruck/part_2.stl; visual mesh filename=package://cybertruck_description/cybertruck/part_2.stl
- added link part_2_2, mass 0.018932239501192930919; collision mesh filename=package://cybertruck_description/cybertruck/part_2.stl; visual mesh filename=package://cybertruck_description/cybertruck/part_2.stl
- added link part_2_3, mass 0.092776419910611848674; collision mesh filename=package://cybertruck_description/cybertruck/part_1.stl; collision mesh filename=package://cybertruck_description/cybertruck/part_2.stl
- added link part_2_4, mass 0.018932239501192930919; collision mesh filename=package://cybertruck_description/cybertruck/part_2.stl; visual mesh filename=package://cybertruck_description/cybertruck/part_2.stl
- link part_1: mass 38.417932880466011625 -> 38.268359742051835326; geometry collision mesh filename=package://cybertruck_description/cybertruck/part_1.stl; collision mesh filename=package://cybertruck_description/cybertruck/part_1.stl
Joints:
- added joint bleft: type revolute, parent part_1, child part_2_4, origin xyz=0.020013294879191026454 0.0019014687469589204062 -0.015010380084460912473 rpy=1.5707963260962891638 -0.65103686779955827202 -1.5707963313037036635, axis 0 0 1, limit effort=1 velocity=20
- added joint fleft: type revolute, parent part_1, child part_2_3, origin xyz=0.020013296253292199578 0.28735142723615747506 -0.075802871142992792053 rpy=1.5707963254239905027 -1.1534217829653337084 -1.5707963304738461474, axis 0 0 1, limit effort=1 velocity=20
- added joint fright: type revolute, parent part_1, child part_2_2, origin xyz=-0.096986703746711311336 0.28735142781322164929 -0.075802871077974356973 rpy=-1.5707963286136721326 1.2602889865366786459 -1.5707963334588699311, axis 0 0 1, limit effort=1 velocity=20
- added joint rightb: type revolute, parent part_1, child part_2, origin xyz=-0.096986705120812491399 0.0019014693240230469244 -0.01501038001944249474 rpy=1.5707963273580198837 -0.16241202732505286011 1.5707963217716685023, axis 0 0 1, limit effort=1 velocity=20

Commit message: reupdated the file

File: cybertruck_description/cybertruck/robot.urdf (robot description, URDF)
Before this commit: robot cybertruck_robot, 5 links, 4 joints
Links:
- removed link part_1
- removed link part_2
- removed link part_2_2
- removed link part_2_3
- removed link part_2_4
- added link carbody, mass 38.268359742051835326; collision mesh filename=package://cybertruck_description/cybertruck/carbody.stl; collision mesh filename=package://cybertruck_description/cybertruck/outerrim.stl
- added link innerrim, mass 0.018932239501192934389; collision mesh filename=package://cybertruck_description/cybertruck/innerrim.stl; visual mesh filename=package://cybertruck_description/cybertruck/innerrim.stl
- added link innerrim_2, mass 0.018932239501192934389; collision mesh filename=package://cybertruck_description/cybertruck/innerrim.stl; visual mesh filename=package://cybertruck_description/cybertruck/innerrim.stl
- added link innerrim_3, mass 0.092776419910611848674; collision mesh filename=package://cybertruck_description/cybertruck/innerrim.stl; collision mesh filename=package://cybertruck_description/cybertruck/outerrim.stl
- added link innerrim_4, mass 0.018932239501192934389; collision mesh filename=package://cybertruck_description/cybertruck/innerrim.stl; visual mesh filename=package://cybertruck_description/cybertruck/innerrim.stl
Joints:
- joint bleft: child part_2_4 -> innerrim_4; parent part_1 -> carbody
- joint fleft: child part_2_3 -> innerrim_3; parent part_1 -> carbody
- joint fright: child part_2_2 -> innerrim_2; parent part_1 -> carbody
- joint rightb: child part_2 -> innerrim; parent part_1 -> carbody
